File: hardware/main/Switches.kicad_sch (KiCad schematic)
At the start: 121 parts, among them J105 Conn_02x03_Odd_Even, Q101 IPT015N10N5, Q102 IPT015N10N5, Q104 IPT015N10N5, Q105 IPT015N10N5, Q107 IPT015N10N5, Q108 IPT015N10N5, Q110 IPT015N10N5, Q111 IPT015N10N5, U101 UCC27211DDAR, U102 UCC27211DDAR, U103 INA823, U104 INA823, U105 INA283, U106 INA283

Commit message: board finalized
Parts:
- removed C105, C106, C113, C114: 100nF, symbol Device:C
- removed C116, C117: 100n, Capacitor_SMD:C_0603_1608Metric_Pad1.08x0.95mm_HandSolder, symbol Device:C_Small
- removed Csn105, Csn107: 100n, Capacitor_SMD:C_1210_3225Metric_Pad1.33x2.70mm_HandSolder, symbol Device:C_Small
- removed Csn106, Csn108: NC, Capacitor_SMD:C_1210_3225Metric_Pad1.33x2.70mm_HandSolder, symbol Device:C_Small
- removed Dsn101, Dsn103, Dsn105, Dsn107: MBR2H100SFT3G, Diode_SMD:D_SOD-123F, symbol Device:D_Schottky_Small
- removed Dsn102, Dsn104, Dsn106, Dsn108: NC, Diode_SMD:D_SOD-123F, symbol Device:D_Schottky_Small
- removed NT101, NT104: NetTie_2, Zenite:NetTie-2_SMD_Pad0.3mm, symbol Device:NetTie_2
- removed NT102, NT103: ~, Zenite:NetTie-2_SMD_Pad0.3mm, symbol Device:NetTie_2
- removed R132, R135: ?, Resistor_SMD:R_0805_2012Metric_Pad1.20x1.40mm_HandSolder, symbol Device:R_Small_US
- removed Rsn105, Rsn107: 10, Resistor_SMD:R_1210_3225Metric_Pad1.30x2.65mm_HandSolder, symbol Device:R_Small_US
- removed Rsn106, Rsn108: NC, Resistor_SMD:R_1210_3225Metric_Pad1.30x2.65mm_HandSolder, symbol Device:R_Small_US
- added Cc410 (x4): 250V 1uF X7R ±10% 20mR 2220, Capacitor_SMD:C_2220_5650Metric, symbol Device:C_Small
- added D405 (x4): SMF100A, Diode_SMD:D_SOD-123F, symbol Diode:SMF18A
- added H105, H106, H107, H108, H109, H110, H111, H112, H113, H114, H115, H116: MountingHole, MountingHole:MountingHole_3.5mm, symbol Mechanical:MountingHole
- added R407 (x4): 0R, Resistor_SMD:R_0805_2012Metric_Pad1.20x1.40mm_HandSolder, symbol Device:R_Small
- C102, C104: footprint Capacitor_SMD:C_0603_1608Metric_Pad1.08x0.95mm_HandSolder -> Capacitor_SMD:C_0805_2012Metric_Pad1.18x1.45mm_HandSolder
- Csn101, Csn103: footprint Capacitor_SMD:C_1210_3225Metric_Pad1.33x2.70mm_HandSolder -> Resistor_SMD:R_1206_3216Metric
- Csn102, Csn104: value NC -> 100n; footprint Capacitor_SMD:C_1210_3225Metric_Pad1.33x2.70mm_HandSolder -> Resistor_SMD:R_1206_3216Metric
- Q101, Q102, Q104, Q105, Q107, Q108, Q110, Q111: value IPT015N10N5 -> BSC093N15NS5; footprint Switches:Infineon_PG-HSOF-8-1_ThermalVias3 -> Zenite:TDSON-8-3; symbol Transistor_FET:IPT015N10N5 -> Device:Q_NMOS_GDS
- Rsn101, Rsn103: footprint Resistor_SMD:R_1210_3225Metric_Pad1.30x2.65mm_HandSolder -> Resistor_SMD:R_1206_3216Metric
- Rsn102, Rsn104: value NC -> 10; footprint Resistor_SMD:R_1210_3225Metric_Pad1.30x2.65mm_HandSolder -> Resistor_SMD:R_1206_3216Metric
- U101, U102: footprint Package_SO:SOIC-8-1EP_3.9x4.9mm_P1.27mm_EP2.514x3.2mm_ThermalVias -> Package_SO:SOIC-8-1EP_3.9x4.9mm_P1.27mm_EP2.514x3.2mm
- U103, U104: footprint Package_SO:VSSOP-8_3.0x3.0mm_P0.65mm -> Package_SO:SOIC-8_3.9x4.9mm_P1.27mm
- U105, U106: footprint (none) -> Package_SO:SOIC-8_3.9x4.9mm_P1.27mm
Connections:
- net Ibat+ is gone; now on net Vbat+_Fus: U105.8 (+)
- net Ibat- is gone; now on net +BATT: U105.1 (-)
- net Imot+ is gone; now on net SL1: U106.8 (+)
- net Imot- is gone; now on net Vout+: U106.1 (-)
- net +5VA: now also C102.1, C104.1, R113.2, R123.1
- net +BATT: now also Q101.2 (D), Q102.2 (D), Q104.2 (D), Q105.2 (D), Cc410.1, Cc410.1, Cc410.1, Cc410.1, R407.1, R407.1; no longer Q101.3 (D), Q102.3 (D), Q104.3 (D), Q105.3 (D), R102.1, R116.1, Rsn102.1, Rsn104.1
- net GND: now also Csn102.2, Csn104.2, Q107.3 (S), Q108.3 (S), Q110.3 (S), Q111.3 (S), Cc410.2, Cc410.2, Cc410.2, Cc410.2, D405.2 (A2), D405.2 (A2); no longer Q107.2 (S), Q108.2 (S), Q110.2 (S), Q111.2 (S), R118.1
- net Iin_Sense: now also U105.5
- net Iout_Sense: now also U106.5
- net SL1: now also Q101.3 (S), Q102.3 (S), Q107.2 (D), Q108.2 (D), Rsn102.1, D405.2 (A2), R407.1; no longer Csn102.2, Q101.2 (S), Q102.2 (S), Q107.3 (D), Q108.3 (D)
- net SL2: now also Q104.3 (S), Q105.3 (S), Q110.2 (D), Q111.2 (D), R118.1, Rsn104.1, D405.2 (A2), R407.1; no longer Csn104.2, Q104.2 (S), Q105.2 (S), Q110.3 (D), Q111.3 (D)
- net Vbat+_Fus: now also R102.1
- net Vin_Sense: now also U103.6; no longer C102.1, R113.1
- net Vout_Sense: now also U104.6; no longer C104.1, R123.1
- net at Csn103.1, Rsn103.2: no longer Csn104.1, Rsn104.2
- net at Csn101.1, Rsn101.2: no longer Csn102.1, Rsn102.2
- net Vout+: now reaches H104.1, R126.1, R129.1
- net Vout+: now also R116.1
- net at R116.2, R119.1, R120.2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: now also R113.1
- net at R123.2: now also R118.2, R120.1, R121.2, U104.2 (-); no longer U104.6
- new net: D405.1 (A1), R407.2 (x4)
- new net: Csn104.1, Rsn104.2
- new net: Csn102.1, Rsn102.2
Other:
- note added: "Control"
- note added: "Fixation"
- note added: "Heatsink"
- moved on the sheet: Rsn101

Commit message: Finalize board sended to faaabrication
Parts:
- H105, H106, H107, H108, H109, H110, H111, H112, H113, H114, H115, H116: footprint MountingHole:MountingHole_3.5mm -> MountingHole:MountingHole_3.5mm_Pad
Changed lines of the file:
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@@
       (effects (font (size 1.27 1.27)) (justify left))
     )
-    (property "Footprint" "MountingHole:MountingHole_3.5mm" (at 186.055 64.77 0)
+    (property "Footprint" "MountingHole:MountingHole_3.5mm_Pad" (at 186.055 64.77 0)
       (effects (font (size 1.27 1.27)) hide)
     )
@@
       (effects (font (size 1.27 1.27)) (justify left))
     )
-    (property "Footprint" "MountingHole:MountingHole_3.5mm" (at 186.055 58.42 0)
+    (property "Footprint" "MountingHole:MountingHole_3.5mm_Pad" (at 186.055 58.42 0)
       (effects (font (size 1.27 1.27)) hide)
     )
@@
       (effects (font (size 1.27 1.27)) (justify left))
     )
-    (property "Footprint" "MountingHole:MountingHole_3.5mm" (at 178.435 58.42 0)
+    (property "Footprint" "MountingHole:MountingHole_3.5mm_Pad" (at 178.435 58.42 0)
       (effects (font (size 1.27 1.27)) hide)
     )
@@
       (effects (font (size 1.27 1.27)) (justify left))
     )
-    (property "Footprint" "MountingHole:MountingHole_3.5mm" (at 185.42 33.655 0)
+    (property "Footprint" "MountingHole:MountingHole_3.5mm_Pad" (at 185.42 33.655 0)
       (effects (font (size 1.27 1.27)) hide)
     )
@@
       (effects (font (size 1.27 1.27)) (justify left))
     )
-    (property "Footprint" "MountingHole:MountingHole_3.5mm" (at 177.8 49.53 0)
+    (property "Footprint" "MountingHole:MountingHole_3.5mm_Pad" (at 177.8 49.53 0)
       (effects (font (size 1.27 1.27)) hide)
     )
@@
       (effects (font (size 1.27 1.27)) (justify left))
     )
-    (property "Footprint" "MountingHole:MountingHole_3.5mm" (at 185.42 27.305 0)
+    (property "Footprint" "MountingHole:MountingHole_3.5mm_Pad" (at 185.42 27.305 0)
       (effects (font (size 1.27 1.27)) hide)
     )
@@
       (effects (font (size 1.27 1.27)) (justify left))
     )
-    (property "Footprint" "MountingHole:MountingHole_3.5mm" (at 177.8 27.305 0)
+    (property "Footprint" "MountingHole:MountingHole_3.5mm_Pad" (at 177.8 27.305 0)
       (effects (font (size 1.27 1.27)) hide)
     )
@@
       (effects (font (size 1.27 1.27)) (justify left))
     )
-    (property "Footprint" "MountingHole:MountingHole_3.5mm" (at 185.42 43.18 0)
+    (property "Footprint" "MountingHole:MountingHole_3.5mm_Pad" (at 185.42 43.18 0)
       (effects (font (size 1.27 1.27)) hide)
     )
@@
       (effects (font (size 1.27 1.27)) (justify left))
     )
-    (property "Footprint" "MountingHole:MountingHole_3.5mm" (at 185.42 49.53 0)
+    (property "Footprint" "MountingHole:MountingHole_3.5mm_Pad" (at 185.42 49.53 0)
       (effects (font (size 1.27 1.27)) hide)
     )
@@
       (effects (font (size 1.27 1.27)) (justify left))
     )
-    (property "Footprint" "MountingHole:MountingHole_3.5mm" (at 177.8 33.655 0)
+    (property "Footprint" "MountingHole:MountingHole_3.5mm_Pad" (at 177.8 33.655 0)
       (effects (font (size 1.27 1.27)) hide)
     )
@@
       (effects (font (size 1.27 1.27)) (justify left))
     )
-    (property "Footprint" "MountingHole:MountingHole_3.5mm" (at 178.435 64.77 0)
+    (property "Footprint" "MountingHole:MountingHole_3.5mm_Pad" (at 178.435 64.77 0)
       (effects (font (size 1.27 1.27)) hide)
     )
@@
       (effects (font (size 1.27 1.27)) (justify left))
     )
-    (property "Footprint" "MountingHole:MountingHole_3.5mm" (at 177.8 43.18 0)
-      (effects (font (size 1.27 1.27)) hide)
-    )
+    (property "Footprint" "MountingHole:MountingHole_3.5mm_Pad" (at 177.8 43.18 0)
+      (effects (font (size 1.27 1.27)) hide)
+    )
